Commit message: Add grid_map as submodule

File: src/ros_unitree/unitree_ros/robots/a1_description/xacro/gazebo.xacro (robot description, xacro)
@@ -69,5 +69,5 @@
                     </horizontal>
                     <vertical> <!-- 30° FOV and 0.5 resolution-->
-                        <samples>61</samples>           <!-- 30° / 0.5° + 1 -->
+                        <samples>60</samples>           <!-- 30° / 0.5° + 1 -->
                         <resolution>1</resolution>
                         <min_angle>-0.2618</min_angle>  <!-- -15° to -->
@@ -76,6 +76,6 @@
                 </scan>
                 <range> <!-- 50 m range -->
-                    <min>0.1</min>
-                    <max>50.0</max>
+                    <min>0.4</min>
+                    <max>50</max>
                     <resolution>0.01</resolution>
                 </range>

File: src/ros_unitree/unitree_ros/robots/a1_description/xacro/robot.xacro (robot description, xacro)
@@ -141,10 +141,10 @@
             <origin xyz="0 0 0.08" rpy="0 0 0"/>
         </visual>
-        <collision>
+        <!-- <collision>
             <geometry>
                 <cylinder length="0.05" radius="0.03"/>
             </geometry>
             <origin xyz="0 0 0.08" rpy="0 0 0"/>
-        </collision>
+        </collision> -->
     </link>
 </robot>

Commit message: Map combiner is added. Submaps are recorded in the maps folder and combined using the map combiner.

File: src/ros_unitree/unitree_ros/robots/a1_description/xacro/gazebo.xacro (robot description, xacro)
@@ -57,5 +57,5 @@
         <material>Gazebo/Red</material>
         <sensor type="gpu_ray" name="lidar_sensor">
-            <pose> 0 0 0.08 0 0 0 </pose>
+            <pose> 0 0 0.15 0 0 0 </pose>
             <visualize>false</visualize>
             <update_rate>10</update_rate> <!-- 10 Hz refresh rate-->
@@ -76,5 +76,5 @@
                 </scan>
                 <range> <!-- 50 m range -->
-                    <min>0.4</min>
+                    <min>0.35</min>
                     <max>50</max>
                     <resolution>0.01</resolution>

File: src/ros_unitree/unitree_ros/robots/a1_description/xacro/robot.xacro (robot description, xacro)
@@ -139,5 +139,5 @@
             </geometry>
             <material name="red"/>
-            <origin xyz="0 0 0.08" rpy="0 0 0"/>
+            <origin xyz="0 0 0.12" rpy="0 0 0"/>
         </visual>
         <!-- <collision>
