Commit message: Octomap and costmap calculations. Move_base integration for autonomous navigation.

File: src/ros_unitree/unitree_ros/robots/a1_description/xacro/robot.xacro (robot description, xacro)
@@ -139,5 +139,5 @@
             </geometry>
             <material name="red"/>
-            <origin xyz="0 0 0.12" rpy="0 0 0"/>
+            <origin xyz="0 0 0.08" rpy="0 0 0"/>
         </visual>
         <!-- <collision>
